Commit message: sim update

File: urdf/cube_stack_arm.xacro (robot description, xacro)
@@ -1,30 +1,14 @@
 <?xml version="1.0"?>
 <robot name="cube_stack_arm" xmlns:xacro="http://ros.org/wiki/xacro">
-  <material name="blue">
-    <color rgba="0 0 0.8 1"/>
-  </material>
-  <material name="black">
-    <color rgba="0 0 0 1"/>
-  </material>
-  <material name="white">
-    <color rgba="1 1 1 1"/>
-  </material>
+  <!-- Attach Arm to Ground -->
   <link name="world"></link>
-  <xacro:include filename="$(find cube_stack_env)/urdf/turtlebot_arm/tbarm.xacro"/>
-  <xacro:turtlebot_arm parent="world" color="White" gripper_color="Green" turtlebot_gripper="true">
+  <xacro:include filename="$(find cube_stack_env)/urdf/turtlebot_arm/turtlebot_arm.xacro"/>
+  <xacro:turtlebot_arm parent="world" color="White" gripper_color="Green" control="effort">
     <origin xyz="0 0 0"/>
   </xacro:turtlebot_arm>
   <xacro:include filename="$(find cube_stack_env)/urdf/sensors.xacro"/>
-  <xacro:depth_camera camera_name="depth_camera" parent_link="arm_base_link">
+  <xacro:depth_camera camera_name="depth_camera" parent_link="arm_base_link" far_range="1.0">
     <box size="0.01 0.01 0.01"/>
-    <origin xyz="0.3 0 0.1" rpy="0 0 3.14"/>
+    <origin xyz="0.6 0 0.1" rpy="0 0 3.14"/>
   </xacro:depth_camera>
-  <!-- Gazebo plugin for ROS Control -->
-  <gazebo>
-    <plugin name="gazebo_ros_control" filename="libgazebo_ros_control.so">
-      <robotNamespace>/cube_stack_arm</robotNamespace>
-      <legacyModeNS>true</legacyModeNS>
-      <robotSimType>gazebo_ros_control/DefaultRobotHWSim</robotSimType>
-    </plugin>
-  </gazebo>
 </robot>

File: urdf/sensors.xacro (robot description, xacro)
@@ -65,5 +65,5 @@
     </gazebo>
   </xacro:macro>
-  <xacro:macro name="depth_camera" params="camera_name parent_link *box *origin">
+  <xacro:macro name="depth_camera" params="camera_name parent_link far_range *box *origin">
     <link name="${camera_name}">
       <collision>
@@ -91,10 +91,10 @@
       <child link="${camera_name}"/>
     </joint>
-    <!-- <link name="camera_depth_link"></link>
+    <link name="camera_depth_link"></link>
     <joint name="camera_depth_joint" type="fixed">
       <origin xyz="0 0 0" rpy="-${pi/2} 0 -${pi/2} "/>
       <parent link="${camera_name}"/>
       <child link="camera_depth_link"/>
-    </joint>     -->
+    </joint>
     <!-- Additional transformation link needed due to frame convention mismatch between gazebo and kinect in rviz
     https://answers.ros.org/question/218395/libgazebo_ros_openni_kinectso-depth-pointcloud-wrong-tf/ -->
@@ -111,5 +111,5 @@
           <clip>
             <near>0.001</near>
-            <far>3</far>
+            <far>${far_range}</far>
           </clip>
         </camera>
@@ -124,7 +124,8 @@
           <depthImageInfoTopicName>/${camera_name}/depth/camera_info</depthImageInfoTopicName>
           <pointCloudTopicName>/${camera_name}/depth/points</pointCloudTopicName>
-          <frameName>${camera_name}</frameName>
+          <frameName>camera_depth_link</frameName>
           <pointCloudCutoff>0.001</pointCloudCutoff>
-          <pointCloudCutoffMax>3.0</pointCloudCutoffMax>
+          <!-- Less then clip range will publish NaN in pointcloud -->
+          <pointCloudCutoffMax>${far_range+1.0}</pointCloudCutoffMax>
           <distortionK1>0.00000001</distortionK1>
           <distortionK2>0.00000001</distortionK2>
@@ -143,21 +144,21 @@
   <xacro:macro name="imu" params="imu_name parent_link *box *origin">
     <link name="${imu_name}">
-<!--       <collision>
-        <origin xyz="0 0 0" rpy="0 0 0"/>
-        <geometry>
-          <xacro:insert_block name="box"/>
-        </geometry>
-      </collision> -->
-      <visual>
-        <origin xyz="0 0 0" rpy="0 0 0"/>
-        <geometry>
-          <xacro:insert_block name="box"/>
-        </geometry>
-      </visual>
-<!--       <inertial>
-        <mass value="0.01" />
-        <origin xyz="0 0 0" rpy="0 0 0"/>
-        <inertia ixx="5.3e-8" ixy="0" ixz="0" iyy="6.7e-9" iyz="0" izz="6.7e-9" />
-      </inertial> -->
+    <!-- <collision>
+      <origin xyz="0 0 0" rpy="0 0 0"/>
+      <geometry>
+        <xacro:insert_block name="box"/>
+      </geometry>
+    </collision> -->
+    <visual>
+      <origin xyz="0 0 0" rpy="0 0 0"/>
+      <geometry>
+        <xacro:insert_block name="box"/>
+      </geometry>
+    </visual>
+    <!-- <inertial>
+      <mass value="0.01" />
+      <origin xyz="0 0 0" rpy="0 0 0"/>
+      <inertia ixx="5.3e-8" ixy="0" ixz="0" iyy="6.7e-9" iyz="0" izz="6.7e-9" />
+    </inertial> -->
     </link>
     <joint name="${imu_name}_joint" type="fixed">

File: urdf/turtlebot_arm/turtlebot_arm.xacro (robot description, xacro)
@@ -3,4 +3,13 @@
 <robot xmlns:xacro="http://ros.org/wiki/xacro">
   <xacro:include filename="$(find cube_stack_env)/urdf/turtlebot_arm/arm_hardware.xacro"/>
+  <xacro:property name="joints_vlimit" value="0.571"/>
+  <xacro:property name="pan_llimit" value="-2.617"/>
+  <xacro:property name="pan_ulimit" value="2.617"/>
+  <xacro:property name="shoulder_llimit" value="-2.617"/>
+  <xacro:property name="shoulder_ulimit" value="2.617"/>
+  <xacro:property name="elbow_llimit" value="-2.617"/>
+  <xacro:property name="elbow_ulimit" value="2.617"/>
+  <xacro:property name="wrist_llimit" value="-1.745"/>
+  <xacro:property name="wrist_ulimit" value="1.745"/>
   <material name="White">
     <color rgba="0.87 0.90 0.87 1.0"/>
@@ -15,5 +24,5 @@
     <color rgba="0.22 0.32 0.14 1.0"/>
   </material>
-  <xacro:macro name="turtlebot_arm" params="parent color turtlebot_gripper gripper_color *origin">
+  <xacro:macro name="turtlebot_arm" params="parent color control gripper_color *origin">
     <link name="arm_base_link"/>
     <joint name="arm_base_joint" type="fixed">
@@ -78,8 +87,45 @@
       <origin xyz="0 0 0" rpy="0 0 0"/>
     </xacro:bioloid_F2_revolute>
-  <!-- gripper - Load Turtlebot gripper -->
-  <xacro:if value="${turtlebot_gripper}">
-  <xacro:include filename="$(find cube_stack_env)/urdf/turtlebot_arm/turtlebot_gripper.xacro"/>
-  </xacro:if>
+    <!-- gripper - Load Turtlebot gripper -->
+    <xacro:include filename="$(find cube_stack_env)/urdf/turtlebot_arm/turtlebot_gripper.xacro"/>
+    <xacro:if value="${control == 'position'}">
+      <xacro:macro name="servo_transmission" params="name">
+        <transmission name="${name}_trans">
+          <type>transmission_interface/SimpleTransmission</type>
+          <actuator name="${name}_motor">
+            <mechanicalReduction>1</mechanicalReduction>
+          </actuator>
+          <joint name="${name}_joint">
+            <hardwareInterface>hardware_interface/PositionJointInterface</hardwareInterface>
+          </joint>
+        </transmission>
+      </xacro:macro>
+    </xacro:if>
+    <xacro:if value="${control == 'effort'}">
+      <xacro:macro name="servo_transmission" params="name">
+        <transmission name="${name}_trans">
+          <type>transmission_interface/SimpleTransmission</type>
+          <actuator name="${name}_motor">
+            <mechanicalReduction>1</mechanicalReduction>
+          </actuator>
+          <joint name="${name}_joint">
+            <hardwareInterface>hardware_interface/EffortJointInterface</hardwareInterface>
+          </joint>
+        </transmission>
+      </xacro:macro>
+    </xacro:if>
+    <xacro:servo_transmission name="arm_shoulder_pan"/>
+    <xacro:servo_transmission name="arm_shoulder_lift"/>
+    <xacro:servo_transmission name="arm_elbow_flex"/>
+    <xacro:servo_transmission name="arm_wrist_flex"/>
+    <xacro:servo_transmission name="gripper"/>
+    <!-- Gazebo plugin for ROS Control -->
+    <gazebo>
+      <plugin name="gazebo_ros_control" filename="libgazebo_ros_control.so">
+        <robotNamespace>/cube_stack_arm</robotNamespace>
+        <legacyModeNS>true</legacyModeNS>
+        <robotSimType>gazebo_ros_control/DefaultRobotHWSim</robotSimType>
+      </plugin>
+    </gazebo>
   </xacro:macro>
 </robot>

Commit message: update
action working
reset working

File: urdf/cube_stack_arm.xacro (robot description, xacro)
@@ -10,5 +10,5 @@
   <xacro:depth_camera camera_name="depth_camera" parent_link="arm_base_link" far_range="1.0">
     <box size="0.01 0.01 0.01"/>
-    <origin xyz="0.6 0 0.1" rpy="0 0 3.14"/>
+    <origin xyz="0.6 0 0.3" rpy="0 0.392 3.14"/>
   </xacro:depth_camera>
 </robot>

File: urdf/sensors.xacro (robot description, xacro)
@@ -101,5 +101,5 @@
     <gazebo reference="${camera_name}">
       <sensor name="${camera_name}_camera" type="depth">
-        <update_rate>20</update_rate>
+        <update_rate>30</update_rate>
         <camera>
           <horizontal_fov>1.047198</horizontal_fov>
@@ -118,5 +118,5 @@
           <alwaysOn>true</alwaysOn>
           <updateRate>1.0</updateRate>
-          <cameraName>${camera_name}_ir</cameraName>
+          <cameraName>${camera_name}</cameraName>
           <imageTopicName>/${camera_name}/rgb/image_raw</imageTopicName>
           <cameraInfoTopicName>/${camera_name}/rgb/camera_info</cameraInfoTopicName>

Commit message: pincher gripper added

File: urdf/cube_stack_arm.xacro (robot description, xacro)
@@ -4,5 +4,5 @@
   <link name="world"></link>
   <xacro:include filename="$(find cube_stack_env)/urdf/turtlebot_arm/turtlebot_arm.xacro"/>
-  <xacro:turtlebot_arm parent="world" color="White" gripper_color="Green" control="effort">
+  <xacro:turtlebot_arm parent="world" color="White" gripper="pincher" control="effort">
     <origin xyz="0 0 0"/>
   </xacro:turtlebot_arm>

File: urdf/turtlebot_arm/arm_hardware.xacro (robot description, xacro)
@@ -291,5 +291,5 @@
     <xacro:macro name="pincher_gripper" params="name color *origin">
       <link name="${name}_link">
-      <xacro:box_inertia length="0.036" width="0.028" height="0.004" mass="0.00001"/>
+      <xacro:box_inertia length="0.036" width="0.028" height="0.004" mass="0.015"/>
       <visual>
         <xacro:insert_block name="origin"/>

File: urdf/turtlebot_arm/turtlebot_arm.xacro (robot description, xacro)
@@ -24,5 +24,5 @@
     <color rgba="0.22 0.32 0.14 1.0"/>
   </material>
-  <xacro:macro name="turtlebot_arm" params="parent color control gripper_color *origin">
+  <xacro:macro name="turtlebot_arm" params="parent color control gripper *origin">
     <link name="arm_base_link"/>
     <joint name="arm_base_joint" type="fixed">
@@ -88,5 +88,10 @@
     </xacro:bioloid_F2_revolute>
     <!-- gripper - Load Turtlebot gripper -->
-    <xacro:include filename="$(find cube_stack_env)/urdf/turtlebot_arm/turtlebot_gripper.xacro"/>
+    <xacro:if value="${gripper == 'turtlebot'}">
+      <xacro:include filename="$(find cube_stack_env)/urdf/turtlebot_arm/turtlebot_gripper.xacro"/>
+    </xacro:if>
+    <xacro:if value="${gripper == 'pincher'}">
+      <xacro:include filename="$(find cube_stack_env)/urdf/turtlebot_arm/pincher_gripper.xacro"/>
+    </xacro:if>
     <xacro:if value="${control == 'position'}">
       <xacro:macro name="servo_transmission" params="name">

File: urdf/turtlebot_arm/turtlebot_gripper.xacro (robot description, xacro)
@@ -39,5 +39,5 @@
       </collision>
     </link>
-    <xacro:finger_fixed parent="gripper_active_link" name="gripper_active_finger" color="${gripper_color}">
+    <xacro:finger_fixed parent="gripper_active_link" name="gripper_active_finger" color="Green">
       <origin xyz="0 0 ${F2_HEIGHT}" rpy="0 0 0"/>
     </xacro:finger_fixed>
@@ -46,5 +46,5 @@
       <origin xyz="0 0 ${-AX12_HEIGHT-F10_HEIGHT+0.001}" rpy="0 ${M_PI} 0"/>
     </xacro:bioloid_F3_fixed>
-    <xacro:finger_fixed parent="gripper_static_link" name="gripper_static_finger" color="${gripper_color}">
+    <xacro:finger_fixed parent="gripper_static_link" name="gripper_static_finger" color="Green">
       <origin xyz="0 0 0" rpy="0 0 ${M_PI}"/>
     </xacro:finger_fixed>
