Commit message: urdf changes

File: urdf/motion_planning/cube_stack.urdf (robot description, URDF)
Before this commit: robot cube_stack_arm, 25 links, 24 joints
Joints:
- joint gripper2_joint: origin xyz=0 0 0 rpy=0 0 0 -> xyz=0 0.04 0 rpy=0 0 0

File: urdf/turtlebot_arm/pincher_gripper.xacro (robot description, xacro)
@@ -24,5 +24,5 @@
     </xacro:pincher_gripper>
     <joint name="gripper2_joint" type="fixed">
-      <origin xyz="0 0 0" rpy="0 0 0"/>
+      <origin xyz="0 0.04 0" rpy="0 0 0"/>
       <axis xyz="1 0 0"/>
       <parent link="gripper_servo_link"/>
@@ -31,5 +31,5 @@
     <!-- Finger 2 -->
     <xacro:pincher_gripper name="gripper_active2" color="Green" >
-      <origin xyz="0.025 0.04 0.0" rpy="${-M_PI/2} 0 0"/>
+      <origin xyz="0.025 0 0.0" rpy="${-M_PI/2} 0 0"/>
     </xacro:pincher_gripper>
     <gazebo reference="gripper_active_link">

Commit message: pick and place partially working

File: urdf/motion_planning/cube_stack.urdf (robot description, URDF)
Before this commit: robot cube_stack_arm, 25 links, 24 joints
Joints:
- joint gripper2_joint: origin xyz=0 0.04 0 rpy=0 0 0 -> xyz=0 0.05 0 rpy=0 0 0

File: urdf/turtlebot_arm/pincher_gripper.xacro (robot description, xacro)
@@ -24,5 +24,5 @@
     </xacro:pincher_gripper>
     <joint name="gripper2_joint" type="fixed">
-      <origin xyz="0 0.04 0" rpy="0 0 0"/>
+      <origin xyz="0 0.05 0" rpy="0 0 0"/>
       <axis xyz="1 0 0"/>
       <parent link="gripper_servo_link"/>
@@ -31,5 +31,5 @@
     <!-- Finger 2 -->
     <xacro:pincher_gripper name="gripper_active2" color="Green" >
-      <origin xyz="0.025 0 0.0" rpy="${-M_PI/2} 0 0"/>
+      <origin xyz="0.025 -0.01 0.0" rpy="${-M_PI/2} 0 0"/>
     </xacro:pincher_gripper>
     <gazebo reference="gripper_active_link">
