Commit message: pick and place mostly working

File: urdf/turtlebot_arm/pincher_gripper.xacro (robot description, xacro)
@@ -15,5 +15,5 @@
       <origin xyz="0 0 0" rpy="0 0 0"/>
       <axis xyz="1 0 0"/>
-      <limit effort="30" velocity="10" lower="-0.01" upper="0.01"/>
+      <limit effort="30" velocity="10" lower="-0.02" upper="0.02"/>
       <parent link="gripper_servo_link"/>
       <child link="gripper_active_link"/>
@@ -31,5 +31,5 @@
     <!-- Finger 2 -->
     <xacro:pincher_gripper name="gripper_active2" color="Green" >
-      <origin xyz="0.025 -0.01 0.0" rpy="${-M_PI/2} 0 0"/>
+      <origin xyz="0.035 -0.01 0.0" rpy="${-M_PI/2} 0 0"/>
     </xacro:pincher_gripper>
     <gazebo reference="gripper_active_link">
